File: air-quality-wing.sch (EAGLE design)
At the start: 37 parts, among them J1 CON-0024, Q1 TR-0001, Q2 TR-0001, Q3 TR-0003, U1 POWER-VREG-FB-EN-SW-350MA, U2 CCS811B-JOPD500, U3 POWER-SWITCH-SIP32509DT, U4 SI7021-A20-GM1R

Commit message: Committing v6 changes:
Changed:

* Formfactor to standard Feather size
* Replaced temperature/humidity sensor with SHTC3
* Replaced TVOC sensor with SGP40
* Changed MCP1640 package to DSON from SOT23-5
* Hatched ground planes on both top and bottom
* Re-designed sensor placement
* Thermal isolation slots for SHTC3
* Pinout for PM2.5 connector reverted back to original design (allows for bidirectional use of cable)

Added:

* Added I2C power control to D4
* Added battery backpack (CR2 holder)
Parts:
- removed JP1, JP4: (no value), microbuilder:HEADER-1X16ROUND
- removed JP2, JP3: (no value), microbuilder:HEADER-1X12
- removed R1, R6, R9: 100k, wolff-den:RES-0041
- removed R4, R5: 20k, wolff-den:RES-0054
- removed U4: SI7021-A20-GM1R, wolff-den:SI7021-A20-GM1R
- added J2: CON-HEADER-1X12-PPPC121LFBN-RC, wolff-den:CON-HEADER-1X12-PPPC121LFBN-RC
- added J3: CON-HEADER-1X16-PPPC161LFBN-RC, wolff-den:CON-HEADER-1X16-PPPC161LFBN-RC
- added JMP1: JUMPER-3/1, wolff-den:JUMPER-3/1
- added PAD1: BH-CR2-1010, wolff-den:BH-CR2-1010
- added SOLDER1: SOLDER, wolff-den:SOLDER-PASTE-ROOM-TEMP-50G
- added U$3, U$4: FIDUCIAL-1MM, wolff-den:FIDUCIAL-1MM
- added U6: IC-SHTC3, wolff-den:IC-SHTC3
- C1, C2: device wolff-den:CAP-0017 -> wolff-den:CAP-0.1U-50V-0402
- C3: device wolff-den:CAP-0010 -> wolff-den:CAP-4.7U-6.3V-0603
- PCB1: value PCB-PS-CCS811-SI7021 -> PCB-PS-AQW; device wolff-den:PCB-PS-CCS811-SI7021 -> wolff-den:PCB-PS-AQW
- R10, R12, R7: device wolff-den:RES-0041 -> wolff-den:RES-100K-1%-0402
- R11: value 1k -> 100k; device wolff-den:RES-1K-1%-0402 -> wolff-den:RES-100K-1%-0402
- R2, R3: value 100k -> 20k; device wolff-den:RES-0041 -> wolff-den:RES-20K-1%-0402
- U$31, U$32: value MOUNTINGHOLE2.5 -> MOUNTING-HOLE-2.5MM-PLATED; device microbuilder:MOUNTINGHOLE2.5 -> wolff-den:MOUNTING-HOLE-2.5MM-PLATED
- U$34, U$35: value FIDUCIAL"" -> FIDUCIAL-1MM; device microbuilder:FIDUCIAL"" -> wolff-den:FIDUCIAL-1MM
- U1: value POWER-VREG-FB-EN-SW-350MA -> POWER-VREG-FB-EN-SW-350MA-DFN8; device wolff-den:POWER-VREG-FB-EN-SW-350MA -> wolff-den:POWER-VREG-FB-EN-SW-350MA-DFN8
- U2: value CCS811B-JOPD500 -> IC-SGP40; device wolff-den:CCS811B-JOPD500 -> wolff-den:IC-SGP40
- U3: value POWER-SWITCH-SIP32509DT -> POWER-SWITCH-SIP32509-SO23-6; device wolff-den:POWER-SWITCH-SIP32509DT -> wolff-den:POWER-SWITCH-SIP32509-SO23-6
- renumbered L2 to FB1
Connections:
- net N$1 renamed V5V0_SW
- net N$3 renamed Q1_D
- net N$6 renamed V5V0_EN
- net N$7 renamed LOAD_SW_EN
- removed net D4: JP2.8, JP3.8
- removed net D5: JP2.7, JP3.7, Q1.G, R10.2, R2.1, R7.2, U2.!RESET
- removed net N$4: R9.2, U2.ADDR
- removed net N$5: U2.PWM, U2.SENSE
- new net D4/SENSORS_VCC: J2.8, JMP1.1
- new net D5/HPMA_EN: J2.7, Q1.G, R10.2, R7.2
- new net SENSORS_VCC: C1.1, C2.1, JMP1.2, R2.2, R3.2, U2.VDD, U2.VDDH, U6.VCC
- net !RESET: now also J3.1; no longer JP1.16, JP4.16
- net +3V3: now also J3.2, JMP1.3; no longer C1.1, C2.1, JP1.15, JP4.15, R2.2, R3.2, R4.2, R5.2, R6.2, U2.VDD, U4.VCC
- net A0: now also J3.5; no longer JP1.12, JP4.12
- net A1: now also J3.6; no longer JP1.11, JP4.11
- net A2: now also J3.7; no longer JP1.10, JP4.10
- net A3: now also J3.8; no longer JP1.9, JP4.9
- net A4: now also J3.9; no longer JP1.8, JP4.8
- net A5: now also J3.10; no longer JP1.7, JP4.7
- net D2: now also J2.10; no longer JP2.10, JP3.10
- net D3: now also J2.9; no longer JP2.9, JP3.9
- net D6: now also J2.6; no longer JP2.6, JP3.6, R3.1, U2.!WAKE
- net D7: now also J2.5; no longer JP2.5, JP3.5
- net D8: now also J2.4; no longer JP2.4, JP3.4, R6.1, U2.!INT
- net EN: now also J2.2; no longer JP2.2, JP3.2
- net GND: now also J1.P$8, J3.4, PAD1.GND, U2.EP, U2.R, U2.VSS, U6.GND; no longer J1.P$1, JP1.13, JP4.13, R1.1, R9.1, U2.EP_GND, U4.GND
- net MD: now also J3.3; no longer JP1.14, JP4.14
- net MISO: now also J3.13; no longer JP1.4, JP4.4
- net MOSI: now also J3.12; no longer JP1.5, JP4.5
- net NC: now also J3.16; no longer JP1.1, JP4.1
- net RX: now also J1.P$6, J3.14; no longer J1.P$3, JP1.3, JP4.3
- net SCK: now also J3.11; no longer JP1.6, JP4.6
- net SCL: now also J2.11, R2.1, U6.SCL; no longer JP2.11, JP3.11, R4.1, U4.SCL
- net SDA: now also J2.12, R3.1, U6.SDA; no longer JP2.12, JP3.12, R5.1, U4.SDA
- net TX: now also J1.P$7, J3.15; no longer J1.P$2, JP1.2, JP4.2
- net V5V0_HAT: now also J1.P$2; no longer J1.P$7
- net VBAT: now also J2.1, PAD1.POS; no longer JP2.1, JP3.1
- net VBUS: now also J2.3; no longer JP2.3, JP3.3, R1.2
Other:
- note added: "I2C Related"
- note added: "Power Supply"
- note added: "SGP40"
- note added: "SHTC3"
- note removed: "Boost"
- note removed: "CSS811"
- note removed: "Si7021"
- moved on the sheet: J1, U1
